File: KiCad/Mic/Mic.kicad_sch (KiCad schematic)
At the start: 27 parts, among them J1 XLR3, J2 1/4" TRS, U1 OPA1641, U2 OPA1641, U3 TS432

Commit message: Minor updates to the scematic and the PCB
Other:
- note added: "68k / 10 k - 9.67 V 47k / 6.8k - 9.81 V"
- note added: "Choose to get about 2+(VCC-2)/2 V DC offset."
- note removed: "Choose to get about (VCC-2)/2 V DC offset."
Changed lines of the file:
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@@
 		)
 	)
-	(text "Choose to get about\n(VCC-2)/2 V DC offset."
+	(text "68k / 10 k - 9.67 V\n47k / 6.8k - 9.81 V"
+		(exclude_from_sim no)
+		(at 166.37 45.72 0)
+		(effects
+			(font
+				(size 1.27 1.27)
+			)
+			(justify right)
+		)
+	)
+	(text "Choose to get about\n2+(VCC-2)/2 V DC offset."
 		(exclude_from_sim no)
 		(at 41.91 27.94 0)
